Commit message: Added odrive control

File: src/ros2_RobotSimulation/PandaRobot/panda_ros2_gazebo/urdf/panda.urdf.xacro (robot description, xacro)
@@ -81,6 +81,8 @@
         <visual>
             <geometry>
-                <mesh filename="file://$(find ur3_ros2_gazebo)/meshes/visual/linear_axis/simplified_static_parts.stl" scale="0.001 0.001 0.001"/>
-            </geometry>
+                <mesh filename="file://$(find ur3_ros2_gazebo)
+                /meshes/visual/linear_axis/simplified_static_parts.stl"
+                scale="0.001 0.001 0.001"/>
+            </geometr
             <material name="Aluminum">
               <color rgba="0.81 0.83 0.85 1.0"/>
@@ -89,5 +91,7 @@
         <collision>
           <geometry>
-            <mesh filename="file://$(find ur3_ros2_gazebo)/meshes/visual/linear_axis/simplified_static_parts.stl" scale="0.001 0.001 0.001"/>
+            <mesh filename="file://$(find ur3_ros2_gazebo)
+            /meshes/visual/linear_axis/simplified_static_parts.stl"
+            scale="0.001 0.001 0.001"/>
           </geometry>
         </collision>
@@ -100,5 +104,7 @@
         <visual>
             <geometry>
-                <mesh filename="file://$(find ur3_ros2_gazebo)/meshes/visual/linear_axis/simplified_dynamic_parts.stl" scale="0.001 0.001 0.001"/>
+                <mesh filename="file://$(find ur3_ros2_gazebo)
+                /meshes/visual/linear_axis/simplified_dynamic_parts.stl"
+                scale="0.001 0.001 0.001"/>
             </geometry>
             <material name="Aluminum_base">
@@ -108,5 +114,7 @@
         <collision>
           <geometry>
-            <mesh filename="file://$(find ur3_ros2_gazebo)/meshes/visual/linear_axis/simplified_dynamic_parts.stl" scale="0.001 0.001 0.001"/>
+            <mesh filename="file://$(find ur3_ros2_gazebo)
+            /meshes/visual/linear_axis/simplified_dynamic_parts.stl"
+            scale="0.001 0.001 0.001"/>
           </geometry>
         </collision>
@@ -120,7 +128,6 @@
     <!-- <child link = "panda_base" /> -->
     <child link = "base_linear_axis" />
-    <origin xyz="0.0 0.0 0.0" rpy="0.0 0.0 0.0" /> <!-- <origin xyz="0.0 0.0 0.65" rpy="0.0 0.0 0.0" /> -->
+    <origin xyz="0.0 0.0 0.0" rpy="0.0 0.0 0.0" />
   </joint>
-cobot_base
   <!-- Linear 7th axis joints -->
   <joint name="base_axis_joint" type="prismatic">

File: src/ros2_RobotSimulation/UniversalRobots/UR3/ur3_ros2_gazebo/urdf/og_ur3.urdf.xacro (robot description, xacro)
@@ -57,6 +57,4 @@
     <!-- Include XACRO-MACRO FILE OF THE UR3 ROBOT -->
     <xacro:include filename="$(find ur3_ros2_gazebo)/urdf/ur3_macro.urdf.xacro" />
-    <!-- Include XACRO-LINEAR AXIS ROS2 CONTROL FILE -->
-    <xacro:include filename="$(find ur3_ros2_gazebo)/urdf/linear_axis_ros2_control.xacro" />
     <!-- Load and initialise UR3 INITIAL POSITIONS FILE:
     <xacro:arg name="initial_positions_file" default="$(find ur3_ros2_gazebo/config/initial_positions.yaml"/>
@@ -76,64 +74,25 @@
     <link name="world"/>
     <link name='ur_base'>
-      <inertial>
-        <origin xyz="0 0 0" rpy="0 0 0"/>
-        <mass value="100"/>
-        <inertia ixx="0.01"  ixy="0"  ixz="0" iyy="0.01" iyz="0" izz="0.01" />
-      </inertial>
-      <collision name='collision'>
-        <origin xyz="0 0 0" rpy=" 0 0 0"/>
-        <geometry>
-          <box size = "0.2 0.2 1.3"/>
-        </geometry>
-      </collision>
-      <visual name='chassis_visual'>
-        <origin xyz="0 0 0" rpy=" 0 0 0"/>
-        <geometry>
-          <box size = "0.2 0.2 1.3"/>
-        </geometry>
-        <material name="red">
-          <color rgba="1 0 0 1"/>
-        </material>
-      </visual>
-    </link>
-    <!-- Linear 7th axis links -->
-    <link name="base_linear_axis">
-        <visual>
-            <geometry>
-                <mesh filename="file://$(find ur3_ros2_gazebo)/meshes/visual/linear_axis/simplified_static_parts.stl" scale="0.001 0.001 0.001"/>
-            </geometry>
-            <material name="Aluminum">
-              <color rgba="0.81 0.83 0.85 1.0"/>
-            </material>
-        </visual>
-        <collision>
-          <geometry>
-            <mesh filename="file://$(find ur3_ros2_gazebo)/meshes/visual/linear_axis/simplified_static_parts.stl" scale="0.001 0.001 0.001"/>
-          </geometry>
-        </collision>
-       <inertial>
-          <mass value="0.5"/>
-         <inertia ixx="0.0" ixy="0.0" ixz="0.0" iyy="0.0" iyz="0.0" izz="0.0"/>
-       </inertial>
-    </link>
-    <link name="cobot_base">
-        <visual>
-            <geometry>
-                <mesh filename="file://$(find ur3_ros2_gazebo)/meshes/visual/linear_axis/simplified_dynamic_parts.stl" scale="0.001 0.001 0.001"/>
-            </geometry>
-            <material name="Aluminum_base">
-              <color rgba="0.57 0.59 0.6 1.0"/>
-            </material>
-        </visual>
-        <collision>
-          <geometry>
-            <mesh filename="file://$(find ur3_ros2_gazebo)/meshes/visual/linear_axis/simplified_dynamic_parts.stl" scale="0.001 0.001 0.001"/>
-          </geometry>
-        </collision>
-       <inertial>
-          <mass value="0.5"/>
-         <inertia ixx="0.002211" ixy="0.0" ixz="0.0" iyy="0.001673" iyz="0.0" izz="0.00387"/>
-       </inertial>
-    </link>
+    <inertial>
+      <origin xyz="0 0 0" rpy="0 0 0"/>
+      <mass value="100"/>
+      <inertia ixx="0.01"  ixy="0"  ixz="0" iyy="0.01" iyz="0" izz="0.01" />
+    </inertial>
+    <collision name='collision'>
+      <origin xyz="0 0 0" rpy=" 0 0 0"/>
+      <geometry>
+        <box size = "0.2 0.2 1.3"/>
+      </geometry>
+    </collision>
+    <visual name='chassis_visual'>
+      <origin xyz="0 0 0" rpy=" 0 0 0"/>
+      <geometry>
+        <box size = "0.2 0.2 1.3"/>
+      </geometry>
+      <material name="red">
+        <color rgba="1 0 0 1"/>
+      </material>
+    </visual>
+  </link>
   <gazebo reference="ur_base">
     <material>Gazebo/Red</material>
@@ -146,19 +105,6 @@
   <joint name="ur_joint" type="fixed">
     <parent link="ur_base" />
-    <child link = "base_linear_axis" />
+    <child link = "base_link" />
     <origin xyz="0.0 0.0 0.655" rpy="0.0 0.0 0.0" />
   </joint>
-  <!-- Linear 7th axis joints -->
-  <joint name="base_axis_joint" type="prismatic">
-        <parent link="base_linear_axis"/>
-        <child link="cobot_base"/>
-        <axis xyz="0 1 0"/>
-        <limit lower="0" upper="0.34" velocity="0.5" effort="1000.0"/>
-        <origin xyz="0 0.16 0" rpy="0 0 3.1415"/>
-  </joint>
-  <joint name="cobot_base-base_link_joint" type="fixed">
-    <parent link="cobot_base" />
-    <child link = "base_link" />
-    <origin xyz="0.0 0.0 0.04" rpy="0.0 0.0 0.0" />
-  </joint>
 </robot>

File: src/ros2_RobotSimulation/UniversalRobots/UR3/ur3_ros2_gazebo/urdf/ur3_macro.urdf.xacro (robot description, xacro)
@@ -61,4 +61,6 @@
   <!-- Load GAZEBO/ROS2_CONTROL file: -->
   <xacro:include filename="$(find ur3_ros2_gazebo)/urdf/ur3_gazebo.xacro" />
+  <!-- Linear axis - ROS2_CONTROL: -->
+  <!-- <xacro:odrive_ros2_control prefix="" name="odrive_ros2_control"/> -->
   <xacro:macro name="ur3_robot" params="
     prefix
