Commit message: Fake hardware function

File: src/ros2_RobotSimulation/UniversalRobots/UR3/ur3_ros2_gazebo/urdf/linear_axis_ros2_control.xacro (robot description, xacro)
@@ -1,18 +1,30 @@
 <?xml version="1.0"?>
 <robot xmlns:xacro="http://www.ros.org/wiki/xacro">
-  <xacro:macro name="odrive_ros2_control"
-    params="prefix name serial_number:=^|000000000000">
+  <xacro:macro name="odrive_ros2_control" params="
+    prefix
+    use_fake_hardware:=false fake_sensor_commands:=false
+    serial_number:=^|000000000000">
     <ros2_control name="BaseAxisControl" type="system">
       <hardware>
-        <plugin>odrive_hardware_interface/ODriveHardwareInterface</plugin>
+        <!-- <plugin>odrive_hardware_interface/ODriveHardwareInterface</plugin> -->
+        <xacro:if value="${use_fake_hardware}">
+          <plugin>fake_components/GenericSystem</plugin>
+          <param name="fake_sensor_commands">${fake_sensor_commands}</param>
+          <param name="state_following_offset">0.0</param>
+        </xacro:if>
+        <xacro:unless value="${use_fake_hardware}">
+          <plugin>gazebo_ros2_control/GazeboSystem</plugin>
+        </xacro:unless>
       </hardware>
-      <sensor name="odrv0">
-        <param name="serial_number">${serial_number}</param>
-      </sensor>
+      <!-- <xacro:unless value="${use_fake_hardware}">
+        <sensor name="odrv0">
+          <param name="serial_number">${serial_number}</param>
+        </sensor>
+      <xacro:unless> -->
       <joint name="${prefix}base_axis_joint">
-        <param name="serial_number">${serial_number}</param>
+        <!-- <param name="serial_number">${serial_number}</param>
         <param name="axis">0</param>
-        <param name="enable_watchdog">0</param>
-        <!-- <command_interface name="position">
+        <param name="enable_watchdog">0</param> -->
+        <command_interface name="position">
           <param name="min">0</param>
           <param name="max">0.34</param>
@@ -24,5 +36,5 @@
         <state_interface name="position"/>
         <state_interface name="velocity"/>
-        <state_interface name="effort"/> -->
+        <state_interface name="effort"/>
       </joint>
     </ros2_control>

File: src/ros2_RobotSimulation/UniversalRobots/UR3/ur3_ros2_gazebo/urdf/ur3.urdf.xacro (robot description, xacro)
@@ -1,62 +1,8 @@
 <?xml version="1.0"?>
-<!--
-# ===================================== COPYRIGHT ===================================== #
-#                                                                                       #
-#  IFRA (Intelligent Flexible Robotics and Assembly) Group, CRANFIELD UNIVERSITY        #
-#  Created on behalf of the IFRA Group at Cranfield University, United Kingdom          #
-#  E-mail: IFRA@cranfield.ac.uk                                                         #
-#                                                                                       #
-#  Licensed under the Apache-2.0 License.                                               #
-#  You may not use this file except in compliance with the License.                     #
-#  You may obtain a copy of the License at: http://www.apache.org/licenses/LICENSE-2.0  #
-#                                                                                       #
-#  Unless required by applicable law or agreed to in writing, software distributed      #
-#  under the License is distributed on an "as-is" basis, without warranties or          #
-#  conditions of any kind, either express or implied. See the License for the specific  #
-#  language governing permissions and limitations under the License.                    #
-#                                                                                       #
-#  IFRA Group - Cranfield University                                                    #
-#  AUTHORS: Mikel Bueno Viso - Mikel.Bueno-Viso@cranfield.ac.uk                         #
-#           Seemal Asif      - s.asif@cranfield.ac.uk                                   #
-#           Phil Webb        - p.f.webb@cranfield.ac.uk                                 #
-#                                                                                       #
-#  Date: July, 2022.                                                                    #
-#                                                                                       #
-# ===================================== COPYRIGHT ===================================== #
-# ===================================== COPYRIGHT ===================================== #
-#                                                                                       #
-#  Some of the information used to build the ROS2 UR3-Robot .urdf files in this ROS2    #
-#  repository has been taken from the following resources:                              #
-#       - Universal Robots ROS2 Description:                                            #
-#         https://github.com/UniversalRobots/Universal_Robots_ROS2_Description          #
-#       - Universal Robots ROS2 Gazebo Simulation:                                      #
-#         https://github.com/UniversalRobots/Universal_Robots_ROS2_Gazebo_Simulation    #
-#                                                                                       #
-#  AUTHORS:                                                                             #
-#       - ROS-Industrial - https://rosindustrial.org                                    #
-#       - Universal Robots - https://github.com/UniversalRobots                         #
-#       - Nadia Hammoudeh Garcia, Kelsey Hawkins, G.A. vd. Hoorn, Lovro Ivanov, Mathias #
-#         Ludtke, Wim Meeussen, Felix Messmer, Miguel Prada Sarasola, Denis Stogl,      #
-#         Andy Zelenak, Marvin Grosse Besselmann.                                       #
-#       - Maintainers: Felix Exner (exner@fzi.de), Tristan Schnell (schnell@fzi.de),    #
-#         Lovro Ivanov (lovro.ivanov@gmail.com), Denis Stogl (denis@stoglrobotics.de).  #
-#                                                                                       #
-#  Copyright (c) 2021, Universal Robots A/S                                             #
-#  (ORIGINAL LICENSE) -> Licensed under the BSD 3-Clause License.                       #
-#                                                                                       #
-#  CHANGES MADE:                                                                        #
-#  Robot information/specifications have been taken, and the code has been modified and #
-#  re-organised in accordance with the ros2_RobotSimulation standards.                  #
-#                                                                                       #
-# ===================================== COPYRIGHT ===================================== #
-# ======= CITE OUR WORK ======= #
-# You can cite our work with the following statement:
-# IFRA (2022) ROS2.0 ROBOT SIMULATION. URL: https://github.com/IFRA-Cranfield/ros2_RobotSimulation.
--->
 <robot xmlns:xacro="http://wiki.ros.org/xacro" name="ur3">
     <!-- Include XACRO-MACRO FILE OF THE UR3 ROBOT -->
     <xacro:include filename="$(find ur3_ros2_gazebo)/urdf/ur3_macro.urdf.xacro" />
     <!-- Include XACRO-LINEAR AXIS ROS2 CONTROL FILE -->
-    <xacro:include filename="$(find ur3_ros2_gazebo)/urdf/linear_axis_ros2_control.xacro" />
+    <!-- <xacro:include filename="$(find ur3_ros2_gazebo)/urdf/linear_axis_ros2_control.xacro" /> -->
     <!-- Load and initialise UR3 INITIAL POSITIONS FILE:
     <xacro:arg name="initial_positions_file" default="$(find ur3_ros2_gazebo/config/initial_positions.yaml"/>
@@ -67,4 +13,8 @@
     <xacro:arg name="safety_pos_margin" default="0.15"/>
     <xacro:arg name="safety_k_position" default="20"/>
+    <!-- Simulation parameters -->
+    <xacro:arg name="use_fake_hardware" default="true" />
+    <xacro:arg name="fake_sensor_commands" default="true" />
+    <xacro:arg name="sim_gazebo" default="false" />
     <!-- Initialise UR3 ROBOT .urdf -->
     <xacro:ur3_robot
@@ -73,5 +23,16 @@
         safety_pos_margin="$(arg safety_pos_margin)"
         safety_k_position="$(arg safety_k_position)"
+        use_fake_hardware="$(arg use_fake_hardware)"
+        fake_sensor_commands="$(arg fake_sensor_commands)"
     />
+    <!-- Gazebo plugins -->
+    <xacro:if value="$(arg sim_gazebo)">
+      <gazebo>
+        <plugin filename="libgazebo_ros2_control.so" name="gazebo_ros2_control">
+          <robot_sim_type>gazebo_ros2_control/GazeboSystem</robot_sim_type>
+          <parameters>$(find ur3_ros2_gazebo)/config/ur3_controller.yaml</parameters>
+        </plugin>
+      </gazebo>
+    </xacro:if>
     <link name="world"/>
     <link name='ur_base'>

File: src/ros2_RobotSimulation/UniversalRobots/UR3/ur3_ros2_gazebo/urdf/ur3_gazebo.xacro (robot description, xacro)
@@ -55,14 +55,41 @@
 -->
 <robot xmlns:xacro="http://www.ros.org/wiki/xacro">
-  <xacro:macro name="ur3_gazebo" params="prefix">
-    <gazebo>
-      <plugin filename="libgazebo_ros2_control.so" name="gazebo_ros2_control">
-        <robot_sim_type>gazebo_ros2_control/GazeboSystem</robot_sim_type>
-        <parameters>$(find ur3_ros2_gazebo)/config/ur3_controller.yaml</parameters>
-      </plugin>
-    </gazebo>
+  <xacro:macro name="ur3_gazebo" params="
+    prefix
+    use_fake_hardware:=false fake_sensor_commands:=false">
+    <ros2_control name="BaseAxisControl" type="system">
+      <hardware>
+        <!-- <plugin>odrive_hardware_interface/ODriveHardwareInterface</plugin> -->
+        <xacro:if value="${use_fake_hardware}">
+          <plugin>fake_components/GenericSystem</plugin>
+          <param name="fake_sensor_commands">${fake_sensor_commands}</param>
+          <param name="state_following_offset">0.0</param>
+        </xacro:if>
+        <xacro:unless value="${use_fake_hardware}">
+          <plugin>gazebo_ros2_control/GazeboSystem</plugin>
+        </xacro:unless>
+      </hardware>
+      <joint name="${prefix}base_axis_joint">
+        <command_interface name="position">
+          <param name="min">0</param>
+          <param name="max">0.34</param>
+        </command_interface>
+        <command_interface name="velocity">
+          <param name="min">-6</param>
+          <param name="max">6</param>
+        </command_interface>
+        <state_interface name="position"/>
+        <state_interface name="velocity"/>
+        <state_interface name="effort"/>
+      </joint>
+    </ros2_control>
     <ros2_control name="GazeboSystem" type="system">
       <hardware>
-        <plugin>gazebo_ros2_control/GazeboSystem</plugin>
+        <xacro:if value="${use_fake_hardware}">
+          <plugin>fake_components/GenericSystem</plugin>
+        </xacro:if>
+        <xacro:unless value="${use_fake_hardware}">
+          <plugin>gazebo_ros2_control/GazeboSystem</plugin>
+        </xacro:unless>
       </hardware>
       <!--
@@ -182,8 +209,8 @@
         <!-- <param name="initial_position">${initial_positions['wrist_3_joint']}</param>   initial position for the FakeSystem -->
       </joint>
-      <joint name="${prefix}base_axis_joint">
-        <command_interface name="position">
-          <param name="min">-0.163</param>
-          <param name="max">0.213</param>
+      <!-- <joint name="${prefix}base_axis_joint">
+        <command_interface name="position">
+          <param name="min">0</param>
+          <param name="max">0.34</param>
         </command_interface>
         <command_interface name="velocity">
@@ -194,5 +221,5 @@
         <state_interface name="velocity"/>
         <state_interface name="effort"/>
-      </joint>
+      </joint> -->
       <!--
       <sensor name="tcp_fts_sensor">

File: src/ros2_RobotSimulation/UniversalRobots/UR3/ur3_ros2_gazebo/urdf/ur3_macro.urdf.xacro (robot description, xacro)
@@ -1,57 +1,3 @@
 <?xml version="1.0"?>
-<!--
-# ===================================== COPYRIGHT ===================================== #
-#                                                                                       #
-#  IFRA (Intelligent Flexible Robotics and Assembly) Group, CRANFIELD UNIVERSITY        #
-#  Created on behalf of the IFRA Group at Cranfield University, United Kingdom          #
-#  E-mail: IFRA@cranfield.ac.uk                                                         #
-#                                                                                       #
-#  Licensed under the Apache-2.0 License.                                               #
-#  You may not use this file except in compliance with the License.                     #
-#  You may obtain a copy of the License at: http://www.apache.org/licenses/LICENSE-2.0  #
-#                                                                                       #
-#  Unless required by applicable law or agreed to in writing, software distributed      #
-#  under the License is distributed on an "as-is" basis, without warranties or          #
-#  conditions of any kind, either express or implied. See the License for the specific  #
-#  language governing permissions and limitations under the License.                    #
-#                                                                                       #
-#  IFRA Group - Cranfield University                                                    #
-#  AUTHORS: Mikel Bueno Viso - Mikel.Bueno-Viso@cranfield.ac.uk                         #
-#           Seemal Asif      - s.asif@cranfield.ac.uk                                   #
-#           Phil Webb        - p.f.webb@cranfield.ac.uk                                 #
-#                                                                                       #
-#  Date: July, 2022.                                                                    #
-#                                                                                       #
-# ===================================== COPYRIGHT ===================================== #
-# ===================================== COPYRIGHT ===================================== #
-#                                                                                       #
-#  Some of the information used to build the ROS2 UR3-Robot .urdf files in this ROS2    #
-#  repository has been taken from the following resources:                              #
-#       - Universal Robots ROS2 Description:                                            #
-#         https://github.com/UniversalRobots/Universal_Robots_ROS2_Description          #
-#       - Universal Robots ROS2 Gazebo Simulation:                                      #
-#         https://github.com/UniversalRobots/Universal_Robots_ROS2_Gazebo_Simulation    #
-#                                                                                       #
-#  AUTHORS:                                                                             #
-#       - ROS-Industrial - https://rosindustrial.org                                    #
-#       - Universal Robots - https://github.com/UniversalRobots                         #
-#       - Nadia Hammoudeh Garcia, Kelsey Hawkins, G.A. vd. Hoorn, Lovro Ivanov, Mathias #
-#         Ludtke, Wim Meeussen, Felix Messmer, Miguel Prada Sarasola, Denis Stogl,      #
-#         Andy Zelenak, Marvin Grosse Besselmann.                                       #
-#       - Maintainers: Felix Exner (exner@fzi.de), Tristan Schnell (schnell@fzi.de),    #
-#         Lovro Ivanov (lovro.ivanov@gmail.com), Denis Stogl (denis@stoglrobotics.de).  #
-#                                                                                       #
-#  Copyright (c) 2021, Universal Robots A/S                                             #
-#  (ORIGINAL LICENSE) -> Licensed under the BSD 3-Clause License.                       #
-#                                                                                       #
-#  CHANGES MADE:                                                                        #
-#  Robot information/specifications have been taken, and the code has been modified and #
-#  re-organised in accordance with the ros2_RobotSimulation standards.                  #
-#                                                                                       #
-# ===================================== COPYRIGHT ===================================== #
-# ======= CITE OUR WORK ======= #
-# You can cite our work with the following statement:
-# IFRA (2022) ROS2.0 ROBOT SIMULATION. URL: https://github.com/IFRA-Cranfield/ros2_RobotSimulation.
--->
 <robot xmlns:xacro="http://wiki.ros.org/xacro">
   <!-- Load PROPERTIES file: -->
@@ -61,11 +7,11 @@
   <!-- Load GAZEBO/ROS2_CONTROL file: -->
   <xacro:include filename="$(find ur3_ros2_gazebo)/urdf/ur3_gazebo.xacro" />
-  <!-- Linear axis - ROS2_CONTROL: -->
-  <!-- <xacro:odrive_ros2_control prefix="" name="odrive_ros2_control"/> -->
   <xacro:macro name="ur3_robot" params="
     prefix
     safety_limits
     safety_pos_margin
-    safety_k_position" >
+    safety_k_position
+    use_fake_hardware:=false
+    fake_sensor_commands:=false">
     <!-- UR3 SPECIFICATIONS/PARAMETERS: -->
     <xacro:ur3_common/>
@@ -73,5 +19,14 @@
     <xacro:ur3_transmission prefix="${prefix}"/>
     <!-- UR3 GAZEBO - ROS2_CONTROL: -->
-    <xacro:ur3_gazebo prefix="${prefix}"/>
+    <xacro:ur3_gazebo
+      prefix="${prefix}"
+      use_fake_hardware="$(arg use_fake_hardware)"
+      fake_sensor_commands="$(arg fake_sensor_commands)"
+      />
+    <!-- <xacro:odrive_ros2_control
+      prefix="${prefix}"
+      use_fake_hardware:="$(arg use_fake_hardware)"
+      fake_sensor_commands:="$(arg fake_sensor_commands)"
+    /> -->
     <!-- ***** UR3 ROBOT .urdf SERIAL CHAIN *****-->
     <!-- Links: -->
